Commit message: update

File: franka_description/robots/common/franka_arm.xacro (robot description, xacro)
@@ -1,9 +1,5 @@
 <?xml version='1.0' encoding='utf-8'?>
 <robot xmlns:xacro="http://www.ros.org/wiki/xacro" name="panda">
-  <xacro:include filename="$(find franka_description)/robots/common/utils.xacro" />
-  <!-- safety_distance: Minimum safety distance in [m] by which the collision volumes are expanded and which is enforced during robot motions -->
-  <!-- arm_id: Namespace of the robot arm. Serves to differentiate between arms in case of multiple instances. -->
-  <!-- joint_limits: description of the joint limits that comes from a YAML file. Example definition: ${xacro.load_yaml('$(find franka_description)/robots/fr3/joint_limits.yaml')} -->
-  <xacro:macro name="franka_arm" params="arm_id:='panda' description_pkg:='franka_description' connected_to:='' xyz:='0 0 0' rpy:='0 0 0' gazebo:=false safety_distance:=0 joint_limits" >
+  <xacro:macro name="franka_arm" params="arm_id:='panda' connected_to:='' xyz:='0 0 0' rpy:='0 0 0' gazebo:=false safety_distance:=0">
     <xacro:unless value="${not connected_to}">
       <joint name="${arm_id}_joint_${connected_to}" type="fixed">
@@ -13,101 +9,53 @@
       </joint>
     </xacro:unless>
-    <xacro:link_with_sc name="link0" gazebo="${gazebo}">
-      <self_collision_geometries>
-        <xacro:collision_capsule xyz="-0.075 0 0.06" direction="x" radius="${0.06+safety_distance}" length="0.03" />
-      </self_collision_geometries>
-    </xacro:link_with_sc>
-    <xacro:link_with_sc name="link1" gazebo="${gazebo}">
-      <self_collision_geometries>
-        <xacro:collision_capsule xyz="0 0 -191.5e-3" radius="${0.06+safety_distance}" length="0.283" />
-      </self_collision_geometries>
-    </xacro:link_with_sc>
+    <!-- 以下、各関節定義 -->
     <joint name="${arm_id}_joint1" type="revolute">
-      <origin rpy="0 0 0" xyz="0 0 0.333" />
-      <parent link="${arm_id}_link0" />
-      <child link="${arm_id}_link1" />
-      <axis xyz="0 0 1" />
-      <xacro:franka-limits name="joint1" config="${joint_limits}" />
-      <dynamics D="1" K="7000" damping="0.003" friction="0.0" mu_coulomb="0" mu_viscous="16" />
+      <origin rpy="0 0 0" xyz="0 0 0.333"/>
+      <parent link="${arm_id}_link0"/>
+      <child link="${arm_id}_link1"/>
+      <axis xyz="0 0 1"/>
+      <limit lower="-2.8973" upper="2.8973" velocity="2.175" effort="87.0"/>
     </joint>
-    <xacro:link_with_sc name="link2" gazebo="${gazebo}">
-      <self_collision_geometries>
-        <xacro:collision_capsule xyz="0 0 0" radius="${0.06+safety_distance}" length="0.12" />
-      </self_collision_geometries>
-    </xacro:link_with_sc>
     <joint name="${arm_id}_joint2" type="revolute">
-      <origin rpy="${-pi/2} 0 0" xyz="0 0 0" />
-      <parent link="${arm_id}_link1" />
-      <child link="${arm_id}_link2" />
-      <axis xyz="0 0 1" />
-      <xacro:franka-limits name="joint2" config="${joint_limits}" />
-      <dynamics D="1" K="7000" damping="0.003" friction="0.0" mu_coulomb="0" mu_viscous="16" />
+      <origin rpy="-1.5707963 0 0" xyz="0 0 0"/>
+      <parent link="${arm_id}_link1"/>
+      <child link="${arm_id}_link2"/>
+      <axis xyz="0 0 1"/>
+      <limit lower="-1.7628" upper="1.7628" velocity="2.175" effort="87.0"/>
     </joint>
-    <xacro:link_with_sc name="link3" gazebo="${gazebo}">
-      <self_collision_geometries>
-        <xacro:collision_capsule xyz="0 0 -0.145" radius="${0.06+safety_distance}" length="0.15" />
-      </self_collision_geometries>
-    </xacro:link_with_sc>
     <joint name="${arm_id}_joint3" type="revolute">
-      <origin rpy="${pi/2} 0 0" xyz="0 -0.316 0" />
-      <parent link="${arm_id}_link2" />
-      <child link="${arm_id}_link3" />
-      <axis xyz="0 0 1" />
-      <xacro:franka-limits name="joint3" config="${joint_limits}" />
-      <dynamics D="1" K="7000" damping="0.003" friction="0.0" mu_coulomb="0" mu_viscous="16" />
+      <origin rpy="1.5707963 0 0" xyz="0 -0.316 0"/>
+      <parent link="${arm_id}_link2"/>
+      <child link="${arm_id}_link3"/>
+      <axis xyz="0 0 1"/>
+      <limit lower="-2.8973" upper="2.8973" velocity="2.175" effort="87.0"/>
     </joint>
-    <xacro:link_with_sc name="link4" gazebo="${gazebo}">
-      <self_collision_geometries>
-        <xacro:collision_capsule xyz="0 0 0" radius="${0.06+safety_distance}" length="0.12" />
-     </self_collision_geometries>
-    </xacro:link_with_sc>
     <joint name="${arm_id}_joint4" type="revolute">
-      <origin rpy="${pi/2} 0 0" xyz="0.0825 0 0" />
-      <parent link="${arm_id}_link3" />
-      <child link="${arm_id}_link4" />
-      <axis xyz="0 0 1" />
-      <xacro:franka-limits name="joint4" config="${joint_limits}" />
-      <dynamics D="1" K="7000" damping="0.003" friction="0.0" mu_coulomb="0" mu_viscous="16" />
+      <origin rpy="1.5707963 0 0" xyz="0.0825 0 0"/>
+      <parent link="${arm_id}_link3"/>
+      <child link="${arm_id}_link4"/>
+      <axis xyz="0 0 1"/>
+      <limit lower="-3.0718" upper="-0.0698" velocity="2.175" effort="87.0"/>
     </joint>
-    <xacro:link_with_sc name="link5" gazebo="${gazebo}">
-      <self_collision_geometries>
-        <xacro:collision_capsule xyz="0 0 -0.26"    radius="${0.060+safety_distance}" length="0.10" />
-        <xacro:collision_capsule xyz="0 0.08 -0.13" radius="${0.025+safety_distance}" length="0.14" />
-      </self_collision_geometries>
-    </xacro:link_with_sc>
     <joint name="${arm_id}_joint5" type="revolute">
-      <origin rpy="${-pi/2} 0 0" xyz="-0.0825 0.384 0" />
-      <parent link="${arm_id}_link4" />
-      <child link="${arm_id}_link5" />
-      <axis xyz="0 0 1" />
-      <xacro:franka-limits name="joint5" config="${joint_limits}" />
-      <dynamics D="1" K="7000" damping="0.003" friction="0.0" mu_coulomb="0" mu_viscous="16" />
+      <origin rpy="-1.5707963 0 0" xyz="-0.0825 0.384 0"/>
+      <parent link="${arm_id}_link4"/>
+      <child link="${arm_id}_link5"/>
+      <axis xyz="0 0 1"/>
+      <limit lower="-2.8973" upper="2.8973" velocity="2.61" effort="12.0"/>
     </joint>
-    <xacro:link_with_sc name="link6" gazebo="${gazebo}">
-      <self_collision_geometries>
-        <xacro:collision_capsule xyz="0 0 -0.03" radius="${0.05+safety_distance}" length="0.08" />
-      </self_collision_geometries>
-    </xacro:link_with_sc>
     <joint name="${arm_id}_joint6" type="revolute">
-      <origin rpy="${pi/2} 0 0" xyz="0 0 0" />
-      <parent link="${arm_id}_link5" />
-      <child link="${arm_id}_link6" />
-      <axis xyz="0 0 1" />
-      <xacro:franka-limits name="joint6" config="${joint_limits}" />
-      <dynamics D="1" K="7000" damping="0.003" friction="0.0" mu_coulomb="0" mu_viscous="16" />
+      <origin rpy="1.5707963 0 0" xyz="0 0 0"/>
+      <parent link="${arm_id}_link5"/>
+      <child link="${arm_id}_link6"/>
+      <axis xyz="0 0 1"/>
+      <limit lower="-0.0175" upper="3.7525" velocity="2.61" effort="12.0"/>
     </joint>
-    <xacro:link_with_sc name="link7" gazebo="${gazebo}" rpy="0 0 ${pi/4}">
-      <self_collision_geometries>
-        <xacro:collision_capsule xyz="0 0 0.01" direction="z" radius="${0.04+safety_distance}" length="0.14" />
-        <xacro:collision_capsule xyz="0.06 0 0.082" direction="x" radius="${0.03+safety_distance}"  length="0.01" />
-      </self_collision_geometries>
-    </xacro:link_with_sc>
     <joint name="${arm_id}_joint7" type="revolute">
-      <origin rpy="${pi/2} 0 0" xyz="0.088 0 0"/>
+      <origin rpy="1.5707963 0 0" xyz="0.088 0 0"/>
       <parent link="${arm_id}_link6"/>
       <child link="${arm_id}_link7"/>
       <axis xyz="0 0 1"/>
-      <xacro:franka-limits name="joint7" config="${joint_limits}" />
-      <dynamics D="1" K="7000" damping="0.003" friction="0.0" mu_coulomb="0" mu_viscous="16"/>
+      <limit lower="-2.8973" upper="2.8973" velocity="2.61" effort="12.0"/>
     </joint>
     <link name="${arm_id}_link8"/>

File: franka_description/robots/common/franka_robot.xacro (robot description, xacro)
@@ -1,10 +1,10 @@
 <?xml version='1.0' encoding='utf-8'?>
 <robot xmlns:xacro="http://www.ros.org/wiki/xacro">
-  <xacro:macro name="franka_robot" params="arm_id joint_limits parent:='world' xyz:='0 0 0' rpy:='0 0 0' hand:=false gazebo:=false tcp_xyz:='0 0 0.1034' tcp_rpy='0 0 0'">
-    <xacro:include filename="$(find franka_description)/robots/common/utils.xacro" />
-    <xacro:include filename="$(find franka_description)/robots/common/franka_arm.xacro" />
-    <xacro:franka_arm arm_id="${arm_id}" safety_distance="0.03" gazebo="${gazebo}" joint_limits="${joint_limits}"/>
+  <xacro:macro name="franka_robot" params="arm_id parent:='world' xyz:='0 0 0' rpy:='0 0 0' hand:=false gazebo:=false tcp_xyz:='0 0 0.1034' tcp_rpy='0 0 0'">
+    <xacro:include filename="/home/shonosukehida/work/PLDM_franka_emika_panda/franka_ros/franka_description/robots/common/utils.xacro" />
+    <xacro:include filename="/home/shonosukehida/work/PLDM_franka_emika_panda/franka_ros/franka_description/robots/common/franka_arm.xacro" />
+    <xacro:franka_arm arm_id="${arm_id}" safety_distance="0.03" gazebo="${gazebo}"/>
     <xacro:if value="${hand}">
-      <xacro:include filename="$(find franka_description)/robots/common/franka_hand.xacro"/>
+      <xacro:include filename="/home/shonosukehida/work/PLDM_franka_emika_panda/franka_ros/franka_description/robots/common/franka_hand.xacro"/>
       <xacro:franka_hand
           arm_id="${arm_id}"

File: franka_description/robots/common/hand.urdf.xacro (robot description, xacro)
@@ -1,5 +1,5 @@
 <?xml version="1.0" encoding="utf-8"?>
 <robot xmlns:xacro="http://www.ros.org/wiki/xacro" name="hand">
-  <xacro:include filename="$(find franka_description)/robots/common/utils.xacro" />
+  <xacro:include filename="/home/shonosukehida/work/PLDM_franka_emika_panda/franka_ros/franka_description/robots/common/utils.xacro" />
   <xacro:include filename="franka_hand.xacro"/>
   <xacro:franka_hand arm_id="panda" safety_distance="0.03"/>

File: franka_description/robots/common/utils.xacro (robot description, xacro)
@@ -2,6 +2,6 @@
 <robot xmlns:xacro="http://www.ros.org/wiki/xacro">
   <!-- Load inertial properties. Property is implicitly passed to macros. -->
-  <xacro:property name="inertial_config" value="$(find franka_description)/robots/common/inertial.yaml"/>
-  <xacro:property name="inertial" value="${xacro.load_yaml(inertial_config)}"/>
+  <!-- <xacro:property name="inertial_config" value="/home/shonosukehida/work/PLDM_franka_emika_panda/franka_ros/franka_description/robots/common/inertial.yaml"/> -->
+  <!-- <xacro:property name="inertial" value="${xacro.load_yaml(inertial_config)}"/> -->
   <!-- ============================================================== -->
   <!-- Macro to add an <inertial> tag based on yaml-load properties   -->
@@ -10,8 +10,7 @@
   <!-- inertial: Dictionary of inertia properties (see inertial.yaml) -->
   <!-- ============================================================== -->
-  <xacro:macro name="inertial_props" params="name inertial:=^">
+  <!-- <xacro:macro name="inertial_props" params="name inertial:=^">
       <xacro:unless value="${name in inertial}">${xacro.warning('No inertia properties defined for: ' + name)}</xacro:unless>
       <xacro:if value="${name in inertial}">
-        <!-- Access inertia properties of link 'name' -->
         <xacro:property name="inertial" value="${inertial[name]}" lazy_eval="false" />
         <inertial>
@@ -22,5 +21,5 @@
         </inertial>
       </xacro:if>
-  </xacro:macro>
+  </xacro:macro> -->
   <!-- ========================================================== -->
   <!-- Macro to add a single link, both with                      -->

File: franka_description/robots/dual_panda/dual_panda_example.urdf.xacro (robot description, xacro)
@@ -3,6 +3,6 @@
   <xacro:arg name="arm_id_1" default="panda_1" />
   <xacro:arg name="arm_id_2" default="panda_2" />
-  <xacro:include filename="$(find franka_description)/robots/common/franka_arm.xacro"/>
-  <xacro:include filename="$(find franka_description)/robots/common/franka_hand.xacro"/>
+  <xacro:include filename="/home/shonosukehida/work/PLDM_franka_emika_panda/franka_ros/franka_description/robots/common/franka_arm.xacro"/>
+  <xacro:include filename="/home/shonosukehida/work/PLDM_franka_emika_panda/franka_ros/franka_description/robots/common/franka_hand.xacro"/>
   <!-- box shaped table as base for the 2 Pandas -->
   <link name="base">
@@ -24,8 +24,8 @@
   </link>
   <!-- right arm with gripper -->
-  <xacro:franka_arm arm_id="$(arg arm_id_1)" connected_to="base"  xyz="0 -0.5 1" safety_distance="0.03" joint_limits="${xacro.load_yaml('$(find franka_description)/robots/panda/joint_limits.yaml')}"/>
+  <xacro:franka_arm arm_id="$(arg arm_id_1)" connected_to="base"  xyz="0 -0.5 1" safety_distance="0.03" />
   <xacro:franka_hand arm_id="$(arg arm_id_1)" rpy="0 0 ${-pi/4}" connected_to="$(arg arm_id_1)_link8" safety_distance="0.03"/>
   <!-- left arm with gripper -->
-  <xacro:franka_arm arm_id="$(arg arm_id_2)" connected_to="base"  xyz="0 0.5 1" safety_distance="0.03" joint_limits="${xacro.load_yaml('$(find franka_description)/robots/panda/joint_limits.yaml')}"/>
+  <xacro:franka_arm arm_id="$(arg arm_id_2)" connected_to="base"  xyz="0 0.5 1" safety_distance="0.03" />
   <xacro:franka_hand arm_id="$(arg arm_id_2)" rpy="0 0 ${-pi/4}" connected_to="$(arg arm_id_2)_link8" safety_distance="0.03"/>
 </robot>

File: franka_description/robots/fr3/fr3.urdf.xacro (robot description, xacro)
@@ -1,5 +1,5 @@
 <?xml version='1.0' encoding='utf-8'?>
 <robot xmlns:xacro="http://www.ros.org/wiki/xacro" name="fr3">
-  <xacro:include filename="$(find franka_description)/robots/common/franka_robot.xacro"/>
+  <xacro:include filename="/home/shonosukehida/work/PLDM_franka_emika_panda/franka_ros/franka_description/robots/common/franka_robot.xacro"/>
   <!-- Name for this robot -->
   <xacro:arg name="arm_id" default="fr3" />
@@ -19,5 +19,4 @@
   <xacro:arg name="rpy" default="0 0 0" />
   <xacro:franka_robot arm_id="$(arg arm_id)"
-                      joint_limits="${xacro.load_yaml('$(find franka_description)/robots/fr3/joint_limits.yaml')}"
                       hand="$(arg hand)"
                       tcp_xyz="$(arg tcp_xyz)"

File: franka_description/robots/panda/panda.urdf.xacro (robot description, xacro)
@@ -1,5 +1,5 @@
 <?xml version='1.0' encoding='utf-8'?>
 <robot xmlns:xacro="http://www.ros.org/wiki/xacro" name="panda">
-  <xacro:include filename="$(find franka_description)/robots/common/franka_robot.xacro"/>
+  <xacro:include filename="/home/shonosukehida/work/PLDM_franka_emika_panda/franka_ros/franka_description/robots/common/franka_robot.xacro"/>
   <!-- Name for this robot -->
   <xacro:arg name="arm_id" default="panda" />
@@ -19,5 +19,4 @@
   <xacro:arg name="rpy" default="0 0 0" />
   <xacro:franka_robot arm_id="$(arg arm_id)"
-                      joint_limits="${xacro.load_yaml('$(find franka_description)/robots/panda/joint_limits.yaml')}"
                       hand="$(arg hand)"
                       tcp_xyz="$(arg tcp_xyz)"

Commit message: update

File: franka_description/robots/common/franka_arm.xacro (robot description, xacro)
@@ -1,5 +1,5 @@
 <?xml version='1.0' encoding='utf-8'?>
 <robot xmlns:xacro="http://www.ros.org/wiki/xacro" name="panda">
-  <xacro:macro name="franka_arm" params="arm_id:='panda' connected_to:='' xyz:='0 0 0' rpy:='0 0 0' gazebo:=false safety_distance:=0">
+  <xacro:macro name="franka_arm" params="arm_id:='panda' connected_to:='' xyz:='0 0 0' rpy:='0 0 0' gazebo:=false safety_distance:=0 inertial:=^">
     <xacro:unless value="${not connected_to}">
       <joint name="${arm_id}_joint_${connected_to}" type="fixed">
@@ -59,10 +59,37 @@
       <limit lower="-2.8973" upper="2.8973" velocity="2.61" effort="12.0"/>
     </joint>
-    <link name="${arm_id}_link8"/>
+    <!-- <link name="${arm_id}_link8"/>
     <joint name="${arm_id}_joint8" type="fixed">
       <origin rpy="0 0 0" xyz="0 0 0.107"/>
       <parent link="${arm_id}_link7"/>
       <child link="${arm_id}_link8"/>
-    </joint>
+    </joint> -->
+    <link name="${arm_id}_link0">
+      <xacro:inertial_props name="${arm_id}_link0" inertial="${inertial}" />
+    </link>
+    <link name="${arm_id}_link1">
+      <xacro:inertial_props name="${arm_id}_link1" inertial="${inertial}" />
+    </link>
+    <link name="${arm_id}_link2">
+      <xacro:inertial_props name="${arm_id}_link2" inertial="${inertial}" />
+    </link>
+    <link name="${arm_id}_link3">
+      <xacro:inertial_props name="${arm_id}_link3" inertial="${inertial}" />
+    </link>
+    <link name="${arm_id}_link4">
+      <xacro:inertial_props name="${arm_id}_link4" inertial="${inertial}" />
+    </link>
+    <link name="${arm_id}_link5">
+      <xacro:inertial_props name="${arm_id}_link5" inertial="${inertial}" />
+    </link>
+    <link name="${arm_id}_link6">
+      <xacro:inertial_props name="${arm_id}_link6" inertial="${inertial}" />
+    </link>
+    <link name="${arm_id}_link7">
+      <xacro:inertial_props name="${arm_id}_link7" inertial="${inertial}" />
+    </link>
+    <link name="${arm_id}_link8">
+      <xacro:inertial_props name="${arm_id}_link8" inertial="${inertial}" />
+    </link>
   </xacro:macro>
 </robot>

File: franka_description/robots/common/franka_robot.xacro (robot description, xacro)
@@ -1,8 +1,9 @@
 <?xml version='1.0' encoding='utf-8'?>
 <robot xmlns:xacro="http://www.ros.org/wiki/xacro">
-  <xacro:macro name="franka_robot" params="arm_id parent:='world' xyz:='0 0 0' rpy:='0 0 0' hand:=false gazebo:=false tcp_xyz:='0 0 0.1034' tcp_rpy='0 0 0'">
+  <xacro:macro name="franka_robot" params="arm_id parent:='world' xyz:='0 0 0' rpy:='0 0 0' hand:=false gazebo:=false tcp_xyz:='0 0 0.1034' tcp_rpy='0 0 0' inertial_path:='$(arg inertial_path)'">
     <xacro:include filename="/home/shonosukehida/work/PLDM_franka_emika_panda/franka_ros/franka_description/robots/common/utils.xacro" />
     <xacro:include filename="/home/shonosukehida/work/PLDM_franka_emika_panda/franka_ros/franka_description/robots/common/franka_arm.xacro" />
-    <xacro:franka_arm arm_id="${arm_id}" safety_distance="0.03" gazebo="${gazebo}"/>
+    <xacro:property name="inertial" value="${xacro.load_yaml(filename=inertial_path)}"/>
+    <xacro:franka_arm arm_id="${arm_id}" safety_distance="0.03" gazebo="${gazebo}" inertial="${inertial}"/>
     <xacro:if value="${hand}">
       <xacro:include filename="/home/shonosukehida/work/PLDM_franka_emika_panda/franka_ros/franka_description/robots/common/franka_hand.xacro"/>

File: franka_description/robots/common/utils.xacro (robot description, xacro)
@@ -10,5 +10,5 @@
   <!-- inertial: Dictionary of inertia properties (see inertial.yaml) -->
   <!-- ============================================================== -->
-  <!-- <xacro:macro name="inertial_props" params="name inertial:=^">
+  <xacro:macro name="inertial_props" params="name inertial:=^">
       <xacro:unless value="${name in inertial}">${xacro.warning('No inertia properties defined for: ' + name)}</xacro:unless>
       <xacro:if value="${name in inertial}">
@@ -21,5 +21,5 @@
         </inertial>
       </xacro:if>
-  </xacro:macro> -->
+  </xacro:macro>
   <!-- ========================================================== -->
   <!-- Macro to add a single link, both with                      -->

File: franka_description/robots/panda/panda.urdf.xacro (robot description, xacro)
@@ -2,4 +2,6 @@
 <robot xmlns:xacro="http://www.ros.org/wiki/xacro" name="panda">
   <xacro:include filename="/home/shonosukehida/work/PLDM_franka_emika_panda/franka_ros/franka_description/robots/common/franka_robot.xacro"/>
+  <!-- inertial YAML のパス -->
+  <xacro:arg name="inertial_path" default="$(find franka_description)/robots/common/inertial.yaml"/>
   <!-- Name for this robot -->
   <xacro:arg name="arm_id" default="panda" />
